Commit message: update modle

File: husky_description/husky_double_welding/r_husky_panda_rviz.urdf (robot description, URDF)
Before this commit: robot husky, 24 links, 23 joints
Links:
- removed link base_footprint
- removed link base_link
- removed link front_bumper_link
- removed link husky_front_left_wheel_link
- removed link husky_front_right_wheel_link
- removed link husky_rear_left_wheel_link
- removed link husky_rear_right_wheel_link
- removed link imu_link
- removed link inertial_link
- removed link panda_link0
- removed link panda_link1
- removed link panda_link2
- removed link panda_link3
- removed link panda_link4
- removed link panda_link5
- removed link panda_link6
- removed link panda_link7
- removed link panda_link8
- removed link rear_bumper_link
- removed link top_chassis_link
- removed link top_plate_front_link
- removed link top_plate_link
- removed link top_plate_rear_link
- removed link user_rail_link
- added link r_base_footprint
- added link r_base_link; collision box size=0.7899200000000001 0.5709 0.10375; collision box size=0.9874 0.5709 0.12375
- added link r_front_bumper_link; visual mesh filename=package://husky_description/meshes/bumper.dae
- added link r_husky_front_left_wheel_link, mass 2.637; collision cylinder length=0.1143 radius=0.1651; visual mesh filename=package://husky_description/meshes/wheel.dae
- added link r_husky_front_right_wheel_link, mass 2.637; collision cylinder length=0.1143 radius=0.1651; visual mesh filename=package://husky_description/meshes/wheel.dae
- added link r_husky_rear_left_wheel_link, mass 2.637; collision cylinder length=0.1143 radius=0.1651; visual mesh filename=package://husky_description/meshes/wheel.dae
- added link r_husky_rear_right_wheel_link, mass 2.637; collision cylinder length=0.1143 radius=0.1651; visual mesh filename=package://husky_description/meshes/wheel.dae
- added link r_imu_link
- added link r_inertial_link, mass 46.034
- added link r_panda_hand, mass 0.73; collision mesh filename=package://franka_panda_description/meshes/collision/hand.stl; visual mesh filename=package://franka_panda_description/meshes/visual/hand.dae
- added link r_panda_leftfinger, mass 0.1; collision mesh filename=package://franka_panda_description/meshes/collision/finger.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; visual mesh filename=package://franka_panda_description/meshes/visual/finger.dae
- added link r_panda_link0; collision mesh filename=package://franka_panda_description/meshes/collision/link0.s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; visual mesh filename=package://franka_panda_description/meshes/visual/link0.dae
- added link r_panda_link1, mass 4.970684; collision mesh filename=package://franka_panda_description/meshes/collision/link1.s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; visual mesh filename=package://franka_panda_description/meshes/visual/link1.dae
- added link r_panda_link2, mass 0.646926; collision mesh filename=package://franka_panda_description/meshes/collision/link2.s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; visual mesh filename=package://franka_panda_description/meshes/visual/link2.dae
- added link r_panda_link3, mass 3.228604; collision mesh filename=package://franka_panda_description/meshes/collision/link3.s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; visual mesh filename=package://franka_panda_description/meshes/visual/link3.dae
- added link r_panda_link4, mass 3.587895; collision mesh filename=package://franka_panda_description/meshes/collision/link4.s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; visual mesh filename=package://franka_panda_description/meshes/visual/link4.dae
- added link r_panda_link5, mass 1.225946; collision mesh filename=package://franka_panda_description/meshes/collision/link5.s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; visual mesh filename=package://franka_panda_description/meshes/visual/link5.dae
- added link r_panda_link6, mass 1.666555; collision mesh filename=package://franka_panda_description/meshes/collision/link6.s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; visual mesh filename=package://franka_panda_description/meshes/visual/link6.dae
- added link r_panda_link7, mass 7.35522e-01; collision mesh filename=package://franka_panda_description/meshes/collision/link7.s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; visual mesh filename=package://franka_panda_description/meshes/visual/link7.dae
- added link r_panda_link8, mass 0.0
- added link r_panda_rightfinger, mass 0.1; collision mesh filename=package://franka_panda_description/meshes/collision/finger.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; visual mesh filename=package://franka_panda_description/meshes/visual/finger.dae
- added link r_rear_bumper_link; visual mesh filename=package://husky_description/meshes/bumper.dae
- added link r_top_chassis_link; visual mesh filename=package://husky_description/meshes/top_chassis.dae
- added link r_top_plate_front_link
- added link r_top_plate_link; collision mesh filename=package://husky_description/meshes/top_plate.stl; visual mesh filename=package://husky_description/meshes/top_plate.dae
- added link r_top_plate_rear_link
- added link r_user_rail_link; visual mesh filename=package://husky_description/meshes/user_rail.dae
Joints:
- removed joint base_footprint_joint
- removed joint front_bumper
- removed joint husky_front_left_wheel
- removed joint husky_front_right_wheel
- removed joint husky_rear_left_wheel
- removed joint husky_rear_right_wheel
- removed joint imu_joint
- removed joint inertial_joint
- removed joint panda_joint1
- removed joint panda_joint2
- removed joint panda_joint3
- removed joint panda_joint4
- removed joint panda_joint5
- removed joint panda_joint6
- removed joint panda_joint7
- removed joint panda_joint8
- removed joint panda_to_world
- removed joint rear_bumper
- removed joint top_chassis_joint
- removed joint top_plate_front_joint
- removed joint top_plate_joint
- removed joint top_plate_rear_joint
- removed joint user_rail
- added joint r_base_footprint_joint: type fixed, parent r_base_link, child r_base_footprint, origin xyz=0 0 -0.13228 rpy=0 0 0
- added joint r_front_bumper: type fixed, parent r_base_link, child r_front_bumper_link, origin xyz=0.48 0 0.091 rpy=0 0 0
- added joint r_husky_front_left_wheel: type revolute, parent r_base_link, child r_husky_front_left_wheel_link, origin xyz=0.256 0.2854 0.03282 rpy=0 0 0, axis 0 1 0, limit lower=-1000 upper=1000 effort=1000 velocity=100
- added joint r_husky_front_right_wheel: type revolute, parent r_base_link, child r_husky_front_right_wheel_link, origin xyz=0.256 -0.2854 0.03282 rpy=0 0 0, axis 0 1 0, limit lower=-1000 upper=1000 effort=1000 velocity=100
- added joint r_husky_rear_left_wheel: type revolute, parent r_base_link, child r_husky_rear_left_wheel_link, origin xyz=-0.256 0.2854 0.03282 rpy=0 0 0, axis 0 1 0, limit lower=-1000 upper=1000 effort=1000 velocity=100
- added joint r_husky_rear_right_wheel: type revolute, parent r_base_link, child r_husky_rear_right_wheel_link, origin xyz=-0.256 -0.2854 0.03282 rpy=0 0 0, axis 0 1 0, limit lower=-1000 upper=1000 effort=1000 velocity=100
- added joint r_imu_joint: type fixed, parent r_base_link, child r_imu_link, origin xyz=0.19 0 0.149 rpy=0 -1.5708 3.1416
- added joint r_inertial_joint: type fixed, parent r_base_link, child r_inertial_link, origin xyz=0 0 0 rpy=0 0 0
- added joint r_panda_finger_joint1: type prismatic, parent r_panda_hand, child r_panda_leftfinger, origin xyz=0 0 0.0584 rpy=0 0 0, axis 0 1 0, limit lower=0.0 upper=0.04 effort=20 velocity=0.2
- added joint r_panda_finger_joint2: type prismatic, parent r_panda_hand, child r_panda_rightfinger, origin xyz=0 0 0.0584 rpy=0 0 0, axis 0 -1 0, limit lower=0.0 upper=0.04 effort=20 velocity=0.2, mimic joint=panda_finger_joint1
- added joint r_panda_hand_joint: type fixed, parent r_panda_link8, child r_panda_hand, origin xyz=0.0 0 0 rpy=0 0 -0.785398163397
- added joint r_panda_joint1: type revolute, parent r_panda_link0, child r_panda_link1, origin xyz=0 0 0.333 rpy=0 0 0, axis 0 0 1, limit lower=-2.8973 upper=2.8973 effort=87 velocity=2.1750
- added joint r_panda_joint2: type revolute, parent r_panda_link1, child r_panda_link2, origin xyz=0 0 0 rpy=-1.57079632679 0 0, axis 0 0 1, limit lower=-1.7628 upper=1.7628 effort=87 velocity=2.1750
- added joint r_panda_joint3: type revolute, parent r_panda_link2, child r_panda_link3, origin xyz=0 -0.316 0 rpy=1.57079632679 0 0, axis 0 0 1, limit lower=-2.8973 upper=2.8973 effort=87 velocity=2.1750
- added joint r_panda_joint4: type revolute, parent r_panda_link3, child r_panda_link4, origin xyz=0.0825 0 0 rpy=1.57079632679 0 0, axis 0 0 1, limit lower=-3.0718 upper=-0.0698 effort=87 velocity=2.1750
- added joint r_panda_joint5: type revolute, parent r_panda_link4, child r_panda_link5, origin xyz=-0.0825 0.384 0 rpy=-1.57079632679 0 0, axis 0 0 1, limit lower=-2.8973 upper=2.8973 effort=12 velocity=2.6100
- added joint r_panda_joint6: type revolute, parent r_panda_link5, child r_panda_link6, origin xyz=0 0 0 rpy=1.57079632679 0 0, axis 0 0 1, limit lower=-0.0175 upper=3.7525 effort=12 velocity=2.6100
- added joint r_panda_joint7: type revolute, parent r_panda_link6, child r_panda_link7, origin xyz=0.088 0 0 rpy=1.57079632679 0 0, axis 0 0 1, limit lower=-2.8973 upper=2.8973 effort=12 velocity=2.6100
- added joint r_panda_joint8: type fixed, parent r_panda_link7, child r_panda_link8, origin xyz=0 0 0.107 rpy=0 0 0, axis 0 0 0
- added joint r_panda_to_world: type fixed, parent r_base_link, child r_panda_link0, origin xyz=0.35 0 0.25 rpy=0 0 0
- added joint r_rear_bumper: type fixed, parent r_base_link, child r_rear_bumper_link, origin xyz=-0.48 0 0.091 rpy=0 0 3.14159
- added joint r_top_chassis_joint: type fixed, parent r_base_link, child r_top_chassis_link
- added joint r_top_plate_front_joint: type fixed, parent r_top_plate_link, child r_top_plate_front_link, origin xyz=0.36367 0 0.00639 rpy=0 0 0
- added joint r_top_plate_joint: type fixed, parent r_base_link, child r_top_plate_link, origin xyz=0.0812 0 0.245 rpy=0 0 0
- added joint r_top_plate_rear_joint: type fixed, parent r_top_plate_link, child r_top_plate_rear_link, origin xyz=-0.36633 0 0.00639 rpy=0 0 0
- added joint r_user_rail: type fixed, parent r_base_link, child r_user_rail_link, origin xyz=0.272 0 0.245 rpy=0 0 0

File: husky_description/husky_single_welding/husky_panda_free.urdf (robot description, URDF)
Before this commit: robot husky, 24 links, 23 joints
Links:
- removed link husky_front_left_wheel_link
- removed link husky_front_right_wheel_link
- removed link husky_rear_left_wheel_link
- removed link husky_rear_right_wheel_link
- added link front_left_wheel_link, mass 2.637; collision cylinder length=0.1143 radius=0.1651; visual mesh filename=package://husky_description/meshes/wheel.dae
- added link front_right_wheel_link, mass 2.637; collision cylinder length=0.1143 radius=0.1651; visual mesh filename=package://husky_description/meshes/wheel.dae
- added link v_t_link
- added link v_x_link
- added link v_y_link
- link base_link: geometry collision box size=0.78992 0.5709 0.10375; collision box size=0.9874 0.5709 0.12375
- link panda_link8: mass None -> 0.0; geometry 
Joints:
- removed joint husky_front_left_wheel
- removed joint husky_front_right_wheel
- removed joint husky_rear_left_wheel
- removed joint husky_rear_right_wheel
- added joint front_left_wheel: type revolute, parent base_link, child front_left_wheel_link, origin xyz=0.0 0.2854 0.03282 rpy=0 0 0, axis 0 -1 0, limit lower=-1000 upper=1000 effort=1000 velocity=100
- added joint front_right_wheel: type revolute, parent base_link, child front_right_wheel_link, origin xyz=0.0 -0.2854 0.03282 rpy=0 0 0, axis 0 1 0, limit lower=-1000 upper=1000 effort=1000 velocity=100
- added joint v_t_joint: type revolute, parent v_t_link, child base_link, origin xyz=0 0 -0.13228 rpy=0 0 0, axis 0 0 1, limit lower=-6.24 upper=6.24 effort=1000.0 velocity=10000.0
- added joint v_x_joint: type prismatic, parent v_x_link, child v_y_link, origin xyz=0 0 -0.13228 rpy=0 0 0, axis 1 0 0, limit lower=-10000.0 upper=-10000.0 effort=1000.0 velocity=10000.0
- added joint v_y_joint: type prismatic, parent v_y_link, child v_t_link, origin xyz=0 0 -0.13228 rpy=0 0 0, axis 0 1 0, limit lower=-10000.0 upper=-10000.0 effort=1000.0 velocity=10000.0
- joint panda_joint8: axis 0 0 1 -> 0 0 0; origin xyz=0.0 0 0.1 rpy=0 0 0 -> xyz=0 0 0.107 rpy=0 0 0
- joint panda_to_world: origin xyz=0.35 0 0.22 rpy=0 0 0 -> xyz=0.35 0 0.25 rpy=0 0 0
