Commit message: change rviz file

File: husky_description/husky_single/husky_panda_rviz.urdf (robot description, URDF)
Before this commit: robot husky, 27 links, 26 joints
Links:
- removed link base_footprint
- removed link base_link
- removed link front_bumper_link
- removed link husky_front_left_wheel_link
- removed link husky_front_right_wheel_link
- removed link husky_rear_left_wheel_link
- removed link husky_rear_right_wheel_link
- removed link imu_link
- removed link inertial_link
- removed link panda_hand
- removed link panda_leftfinger
- removed link panda_link0
- removed link panda_link1
- removed link panda_link2
- removed link panda_link3
- removed link panda_link4
- removed link panda_link5
- removed link panda_link6
- removed link panda_link7
- removed link panda_link8
- removed link panda_rightfinger
- removed link rear_bumper_link
- removed link top_chassis_link
- removed link top_plate_front_link
- removed link top_plate_link
- removed link top_plate_rear_link
- removed link user_rail_link
- added link rviz_base_footprint
- added link rviz_base_link; collision box size=0.7899200000000001 0.5709 0.10375; collision box size=0.9874 0.5709 0.12375
- added link rviz_front_bumper_link; visual mesh filename=package://husky_description/meshes/bumper.dae
- added link rviz_husky_front_left_wheel_link, mass 2.637; collision cylinder length=0.1143 radius=0.1651; visual mesh filename=package://husky_description/meshes/wheel.dae
- added link rviz_husky_front_right_wheel_link, mass 2.637; collision cylinder length=0.1143 radius=0.1651; visual mesh filename=package://husky_description/meshes/wheel.dae
- added link rviz_husky_rear_left_wheel_link, mass 2.637; collision cylinder length=0.1143 radius=0.1651; visual mesh filename=package://husky_description/meshes/wheel.dae
- added link rviz_husky_rear_right_wheel_link, mass 2.637; collision cylinder length=0.1143 radius=0.1651; visual mesh filename=package://husky_description/meshes/wheel.dae
- added link rviz_imu_link
- added link rviz_inertial_link, mass 46.034
- added link rviz_panda_hand, mass 0.73; collision mesh filename=package://franka_panda_description/meshes/collision/hand.stl; visual mesh filename=package://franka_panda_description/meshes/visual/hand.dae
- added link rviz_panda_leftfinger, mass 0.1; collision mesh filename=package://franka_panda_description/meshes/collision/finger.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; visual mesh filename=package://franka_panda_description/meshes/visual/finger.dae
- added link rviz_panda_link0; collision mesh filename=package://franka_panda_description/meshes/collision/link0.s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; visual mesh filename=package://franka_panda_description/meshes/visual/link0.dae
- added link rviz_panda_link1, mass 4.970684; collision mesh filename=package://franka_panda_description/meshes/collision/link1.s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; visual mesh filename=package://franka_panda_description/meshes/visual/link1.dae
- added link rviz_panda_link2, mass 0.646926; collision mesh filename=package://franka_panda_description/meshes/collision/link2.s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; visual mesh filename=package://franka_panda_description/meshes/visual/link2.dae
- added link rviz_panda_link3, mass 3.228604; collision mesh filename=package://franka_panda_description/meshes/collision/link3.s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; visual mesh filename=package://franka_panda_description/meshes/visual/link3.dae
- added link rviz_panda_link4, mass 3.587895; collision mesh filename=package://franka_panda_description/meshes/collision/link4.s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; visual mesh filename=package://franka_panda_description/meshes/visual/link4.dae
- added link rviz_panda_link5, mass 1.225946; collision mesh filename=package://franka_panda_description/meshes/collision/link5.s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; visual mesh filename=package://franka_panda_description/meshes/visual/link5.dae
- added link rviz_panda_link6, mass 1.666555; collision mesh filename=package://franka_panda_description/meshes/collision/link6.s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; visual mesh filename=package://franka_panda_description/meshes/visual/link6.dae
- added link rviz_panda_link7, mass 7.35522e-01; collision mesh filename=package://franka_panda_description/meshes/collision/link7.s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; visual mesh filename=package://franka_panda_description/meshes/visual/link7.dae
- added link rviz_panda_link8, mass 0.0
- added link rviz_panda_rightfinger, mass 0.1; collision mesh filename=package://franka_panda_description/meshes/collision/finger.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; visual mesh filename=package://franka_panda_description/meshes/visual/finger.dae
- added link rviz_rear_bumper_link; visual mesh filename=package://husky_description/meshes/bumper.dae
- added link rviz_top_chassis_link; visual mesh filename=package://husky_description/meshes/top_chassis.dae
- added link rviz_top_plate_front_link
- added link rviz_top_plate_link; collision mesh filename=package://husky_description/meshes/top_plate.stl; visual mesh filename=package://husky_description/meshes/top_plate.dae
- added link rviz_top_plate_rear_link
- added link rviz_user_rail_link; visual mesh filename=package://husky_description/meshes/user_rail.dae
Joints:
- joint base_footprint_joint: child base_footprint -> rviz_base_footprint; parent base_link -> rviz_base_link
- joint front_bumper: child front_bumper_link -> rviz_front_bumper_link; parent base_link -> rviz_base_link
- joint husky_front_left_wheel: child husky_front_left_wheel_link -> rviz_husky_front_left_wheel_link; parent base_link -> rviz_base_link
- joint husky_front_right_wheel: child husky_front_right_wheel_link -> rviz_husky_front_right_wheel_link; parent base_link -> rviz_base_link
- joint husky_rear_left_wheel: child husky_rear_left_wheel_link -> rviz_husky_rear_left_wheel_link; parent base_link -> rviz_base_link
- joint husky_rear_right_wheel: child husky_rear_right_wheel_link -> rviz_husky_rear_right_wheel_link; parent base_link -> rviz_base_link
- joint imu_joint: child imu_link -> rviz_imu_link; parent base_link -> rviz_base_link
- joint inertial_joint: child inertial_link -> rviz_inertial_link; parent base_link -> rviz_base_link
- joint panda_finger_joint1: child panda_leftfinger -> rviz_panda_leftfinger; parent panda_hand -> rviz_panda_hand
- joint panda_finger_joint2: child panda_rightfinger -> rviz_panda_rightfinger; parent panda_hand -> rviz_panda_hand
- joint panda_hand_joint: child panda_hand -> rviz_panda_hand; parent panda_link8 -> rviz_panda_link8
- joint panda_joint1: child panda_link1 -> rviz_panda_link1; parent panda_link0 -> rviz_panda_link0
- joint panda_joint2: child panda_link2 -> rviz_panda_link2; parent panda_link1 -> rviz_panda_link1
- joint panda_joint3: child panda_link3 -> rviz_panda_link3; parent panda_link2 -> rviz_panda_link2
- joint panda_joint4: child panda_link4 -> rviz_panda_link4; parent panda_link3 -> rviz_panda_link3
- joint panda_joint5: child panda_link5 -> rviz_panda_link5; parent panda_link4 -> rviz_panda_link4
- joint panda_joint6: child panda_link6 -> rviz_panda_link6; parent panda_link5 -> rviz_panda_link5
- joint panda_joint7: child panda_link7 -> rviz_panda_link7; parent panda_link6 -> rviz_panda_link6
- joint panda_joint8: child panda_link8 -> rviz_panda_link8; parent panda_link7 -> rviz_panda_link7
- joint panda_to_world: child panda_link0 -> rviz_panda_link0; parent base_link -> rviz_base_link
- joint rear_bumper: child rear_bumper_link -> rviz_rear_bumper_link; parent base_link -> rviz_base_link
- joint top_chassis_joint: child top_chassis_link -> rviz_top_chassis_link; parent base_link -> rviz_base_link
- joint top_plate_front_joint: child top_plate_front_link -> rviz_top_plate_front_link; parent top_plate_link -> rviz_top_plate_link
- joint top_plate_joint: child top_plate_link -> rviz_top_plate_link; parent base_link -> rviz_base_link
- joint top_plate_rear_joint: child top_plate_rear_link -> rviz_top_plate_rear_link; parent top_plate_link -> rviz_top_plate_link
- joint user_rail: child user_rail_link -> rviz_user_rail_link; parent base_link -> rviz_base_link

Commit message: update velodyne modle

File: husky_description/husky_single/husky_panda_rviz.urdf (robot description, URDF)
Before this commit: robot husky, 27 links, 26 joints
Links:
- added link velodyne; visual mesh filename=package://velodyne_description/meshes/VLP16_base_1.dae; visual mesh filename=package://velodyne_description/meshes/VLP16_base_2.dae
Joints:
- added joint velodyne_joint: type fixed, parent rviz_base_link, child velodyne, origin xyz=-0.2 0 0.75 rpy=0 0 0
