Commit message: add 2f_85 gripper

File: husky_description/husky_single/husky_panda_2f_85_rviz_ns1.urdf (robot description, URDF)
Before this commit: robot ns1_husky, 27 links, 26 joints
Links:
- removed link ns1_rviz_panda_hand
- removed link ns1_rviz_panda_leftfinger
- removed link ns1_rviz_panda_rightfinger
- added link ns1_left_inner_finger, mass 0.00724255346165745; collision mesh filename=package://kimm_robotiq_2f_85_description/meshes_aprice/inne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; visual mesh filename=package://kimm_robotiq_2f_85_description/meshes_aprice/inne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
- added link ns1_left_inner_knuckle, mass 0.0110930853895903; collision mesh filename=package://kimm_robotiq_2f_85_description/meshes_aprice/inne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; visual mesh filename=package://kimm_robotiq_2f_85_description/meshes_aprice/inne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
- added link ns1_left_outer_finger, mass 0.0273093985570947; collision mesh filename=package://kimm_robotiq_2f_85_description/meshes_aprice/oute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; visual mesh filename=package://kimm_robotiq_2f_85_description/meshes_aprice/oute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
- added link ns1_left_outer_knuckle, mass 0.00684838849434396; collision mesh filename=package://kimm_robotiq_2f_85_description/meshes_aprice/oute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; visual mesh filename=package://kimm_robotiq_2f_85_description/meshes_aprice/oute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
- added link ns1_right_inner_finger, mass 0.00724255346165744; collision mesh filename=package://kimm_robotiq_2f_85_description/meshes_aprice/inne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; visual mesh filename=package://kimm_robotiq_2f_85_description/meshes_aprice/inne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
- added link ns1_right_inner_knuckle, mass 0.0110930853895903; collision mesh filename=package://kimm_robotiq_2f_85_description/meshes_aprice/inne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; visual mesh filename=package://kimm_robotiq_2f_85_description/meshes_aprice/inne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
- added link ns1_right_outer_finger, mass 0.0273093985570947; collision mesh filename=package://kimm_robotiq_2f_85_description/meshes_aprice/oute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; visual mesh filename=package://kimm_robotiq_2f_85_description/meshes_aprice/oute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
- added link ns1_right_outer_knuckle, mass 0.00684838849401352; collision mesh filename=package://kimm_robotiq_2f_85_description/meshes_aprice/oute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; visual mesh filename=package://kimm_robotiq_2f_85_description/meshes_aprice/oute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
- added link ns1_robotiq_85_base_link, mass 0.30915; collision mesh filename=package://kimm_robotiq_2f_85_description/meshes_aprice/robo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; visual mesh filename=package://kimm_robotiq_2f_85_description/meshes_aprice/robo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
Joints:
- removed joint ns1_panda_finger_joint1
- removed joint ns1_panda_finger_joint2
- removed joint ns1_panda_hand_joint
- added joint ns1_finger_joint: type revolute, parent ns1_robotiq_85_base_link, child ns1_left_outer_knuckle, origin xyz=0.0306011444260539 0 0.0627920162695395 rpy=0 0 0, axis 0 -1 0, limit lower=0 upper=0.725 effort=1000 velocity=2.0
- added joint ns1_left_inner_finger_joint: type revolute, parent ns1_left_inner_knuckle, child ns1_left_inner_finger, origin xyz=0.034585310861294 0 0.0454970193817975 rpy=0 0 0, axis 0 -1 0, limit lower=0 upper=0.8757 effort=1000 velocity=2.0, mimic joint=finger_joint multiplier=-1 offset=0
- added joint ns1_left_inner_knuckle_joint: type revolute, parent ns1_robotiq_85_base_link, child ns1_left_inner_knuckle, origin xyz=0.0127000000001501 0 0.0693074999999639 rpy=0 0 0, axis 0 -1 0, limit lower=0 upper=0.8757 effort=1000 velocity=2.0, mimic joint=finger_joint multiplier=1 offset=0
- added joint ns1_left_outer_finger_joint: type fixed, parent ns1_left_outer_knuckle, child ns1_left_outer_finger, origin xyz=0.0316910442266543 0 -0.00193396375724605 rpy=0 0 0, axis 0 -1 0
- added joint ns1_panda_robotiq_attachment_joint: type fixed, parent ns1_rviz_panda_link8, child ns1_robotiq_85_base_link, origin xyz=0 0 0 rpy=0 0 1.5707963268, axis 0 0 0
- added joint ns1_right_inner_finger_joint: type revolute, parent ns1_right_inner_knuckle, child ns1_right_inner_finger, origin xyz=0.0341060475457406 0 0.0458573878541688 rpy=0 0 0, axis 0 1 0, limit lower=0 upper=0.8757 effort=1000 velocity=2.0, mimic joint=finger_joint multiplier=1 offset=0
- added joint ns1_right_inner_knuckle_joint: type revolute, parent ns1_robotiq_85_base_link, child ns1_right_inner_knuckle, origin xyz=-0.0126999999998499 0 0.0693075000000361 rpy=0 0 3.14159265358979, axis 0 1 0, limit lower=0 upper=0.8757 effort=1000 velocity=2.0, mimic joint=finger_joint multiplier=-1 offset=0
- added joint ns1_right_outer_finger_joint: type fixed, parent ns1_right_outer_knuckle, child ns1_right_outer_finger, origin xyz=0.0317095909367246 0 -0.0016013564954687 rpy=0 0 0, axis 0 1 0
- added joint ns1_right_outer_knuckle_joint: type revolute, parent ns1_robotiq_85_base_link, child ns1_right_outer_knuckle, origin xyz=-0.0306011444258893 0 0.0627920162695395 rpy=0 0 3.14159265358979, axis 0 1 0, limit lower=0 upper=0.8757 effort=1000 velocity=2.0, mimic joint=finger_joint multiplier=-1 offset=0

File: husky_description/husky_single/husky_panda_hand_free.urdf (robot description, URDF)
Before this commit: robot husky, 28 links, 27 joints
Links:
- removed link husky_right_left_wheel_link
- added link husky_front_right_wheel_link, mass 2.637; collision cylinder length=0.1143 radius=0.1651; visual mesh filename=package://husky_description/meshes/wheel.dae
Joints:
- removed joint husky_right_left_wheel
- added joint husky_front_right_wheel: type revolute, parent base_link, child husky_front_right_wheel_link, origin xyz=0.0 -0.2854 0.03282 rpy=0 0 0, axis 0 1 0, limit lower=-1000 upper=1000 effort=1000 velocity=100
- joint v_t_joint: origin xyz=0 0 -0.13228 rpy=0 0 0 -> xyz=0 0 0.0 rpy=0 0 0
- joint v_x_joint: origin xyz=0 0 -0.13228 rpy=0 0 0 -> xyz=0 0 0.0 rpy=0 0 0
- joint v_y_joint: origin xyz=0 0 -0.13228 rpy=0 0 0 -> xyz=0 0 0.0 rpy=0 0 0
