Commit message: add robotiq gripper to husky_panda urdf

File: husky_description/husky_single/husky_panda_2f_85.urdf (robot description, URDF)
Before this commit: robot ns1_husky, 33 links, 32 joints
Links:
- removed link ns1_left_inner_finger
- removed link ns1_left_inner_knuckle
- removed link ns1_left_outer_finger
- removed link ns1_left_outer_knuckle
- removed link ns1_right_inner_finger
- removed link ns1_right_inner_knuckle
- removed link ns1_right_outer_finger
- removed link ns1_right_outer_knuckle
- removed link ns1_robotiq_85_base_link
- removed link ns1_rviz_base_footprint
- removed link ns1_rviz_base_link
- removed link ns1_rviz_front_bumper_link
- removed link ns1_rviz_husky_front_left_wheel_link
- removed link ns1_rviz_husky_front_right_wheel_link
- removed link ns1_rviz_husky_rear_left_wheel_link
- removed link ns1_rviz_husky_rear_right_wheel_link
- removed link ns1_rviz_imu_link
- removed link ns1_rviz_inertial_link
- removed link ns1_rviz_panda_link0
- removed link ns1_rviz_panda_link1
- removed link ns1_rviz_panda_link2
- removed link ns1_rviz_panda_link3
- removed link ns1_rviz_panda_link4
- removed link ns1_rviz_panda_link5
- removed link ns1_rviz_panda_link6
- removed link ns1_rviz_panda_link7
- removed link ns1_rviz_panda_link8
- removed link ns1_rviz_rear_bumper_link
- removed link ns1_rviz_top_chassis_link
- removed link ns1_rviz_top_plate_front_link
- removed link ns1_rviz_top_plate_link
- removed link ns1_rviz_top_plate_rear_link
- removed link ns1_rviz_user_rail_link
- added link base_footprint
- added link base_link; collision box size=0.78992 0.5709 0.10375; collision box size=0.9874 0.5709 0.12375
- added link front_bumper_link; visual mesh filename=package://husky_description/meshes/bumper.dae
- added link husky_front_left_wheel_link, mass 2.637; collision cylinder length=0.1143 radius=0.1651; visual mesh filename=package://husky_description/meshes/wheel.dae
- added link husky_front_right_wheel_link, mass 2.637; collision cylinder length=0.1143 radius=0.1651; visual mesh filename=package://husky_description/meshes/wheel.dae
- added link imu_link
- added link inertial_link, mass 46.034
- added link left_inner_finger, mass 0.00724255346165745; collision mesh filename=package://kimm_robotiq_2f_85_description/meshes_aprice/inne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; visual mesh filename=package://kimm_robotiq_2f_85_description/meshes_aprice/inne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
- added link left_inner_knuckle, mass 0.0110930853895903; collision mesh filename=package://kimm_robotiq_2f_85_description/meshes_aprice/inne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; visual mesh filename=package://kimm_robotiq_2f_85_description/meshes_aprice/inne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
- added link left_outer_finger, mass 0.0273093985570947; collision mesh filename=package://kimm_robotiq_2f_85_description/meshes_aprice/oute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; visual mesh filename=package://kimm_robotiq_2f_85_description/meshes_aprice/oute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
- added link left_outer_knuckle, mass 0.00684838849434396; collision mesh filename=package://kimm_robotiq_2f_85_description/meshes_aprice/oute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; visual mesh filename=package://kimm_robotiq_2f_85_description/meshes_aprice/oute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
- added link panda_link0; collision mesh filename=package://franka_panda_description/meshes/collision/link0.s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; visual mesh filename=package://franka_panda_description/meshes/visual/link0.dae
- added link panda_link1, mass 4.970684; collision mesh filename=package://franka_panda_description/meshes/collision/link1.s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; visual mesh filename=package://franka_panda_description/meshes/visual/link1.dae
- added link panda_link2, mass 0.646926; collision mesh filename=package://franka_panda_description/meshes/collision/link2.s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; visual mesh filename=package://franka_panda_description/meshes/visual/link2.dae
- added link panda_link3, mass 3.228604; collision mesh filename=package://franka_panda_description/meshes/collision/link3.s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; visual mesh filename=package://franka_panda_description/meshes/visual/link3.dae
- added link panda_link4, mass 3.587895; collision mesh filename=package://franka_panda_description/meshes/collision/link4.s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; visual mesh filename=package://franka_panda_description/meshes/visual/link4.dae
- added link panda_link5, mass 1.225946; collision mesh filename=package://franka_panda_description/meshes/collision/link5.s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; visual mesh filename=package://franka_panda_description/meshes/visual/link5.dae
- added link panda_link6, mass 1.666555; collision mesh filename=package://franka_panda_description/meshes/collision/link6.s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; visual mesh filename=package://franka_panda_description/meshes/visual/link6.dae
- added link panda_link7, mass 7.35522e-01; collision mesh filename=package://franka_panda_description/meshes/collision/link7.s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; visual mesh filename=package://franka_panda_description/meshes/visual/link7.dae
- added link panda_link8, mass 0.0
- added link rear_bumper_link; visual mesh filename=package://husky_description/meshes/bumper.dae
- added link right_inner_finger, mass 0.00724255346165744; collision mesh filename=package://kimm_robotiq_2f_85_description/meshes_aprice/inne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; visual mesh filename=package://kimm_robotiq_2f_85_description/meshes_aprice/inne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
- added link right_inner_knuckle, mass 0.0110930853895903; collision mesh filename=package://kimm_robotiq_2f_85_description/meshes_aprice/inne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; visual mesh filename=package://kimm_robotiq_2f_85_description/meshes_aprice/inne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
- added link right_outer_finger, mass 0.0273093985570947; collision mesh filename=package://kimm_robotiq_2f_85_description/meshes_aprice/oute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; visual mesh filename=package://kimm_robotiq_2f_85_description/meshes_aprice/oute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
- added link right_outer_knuckle, mass 0.00684838849401352; collision mesh filename=package://kimm_robotiq_2f_85_description/meshes_aprice/oute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; visual mesh filename=package://kimm_robotiq_2f_85_description/meshes_aprice/oute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
- added link robotiq_85_base_link, mass 0.79501; collision mesh filename=package://kimm_robotiq_2f_85_description/meshes_aprice/robo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; visual mesh filename=package://kimm_robotiq_2f_85_description/meshes_aprice/robo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
- added link top_chassis_link; visual mesh filename=package://husky_description/meshes/top_chassis.dae
- added link top_plate_front_link
- added link top_plate_link; collision mesh filename=package://husky_description/meshes/top_plate.stl; visual mesh filename=package://husky_description/meshes/top_plate.dae
- added link top_plate_rear_link
- added link user_rail_link; visual mesh filename=package://husky_description/meshes/user_rail.dae
- added link v_t_link
- added link v_x_link
- added link v_y_link
Joints:
- removed joint ns1_base_footprint_joint
- removed joint ns1_finger_joint
- removed joint ns1_front_bumper
- removed joint ns1_husky_front_left_wheel
- removed joint ns1_husky_front_right_wheel
- removed joint ns1_husky_rear_left_wheel
- removed joint ns1_husky_rear_right_wheel
- removed joint ns1_imu_joint
- removed joint ns1_inertial_joint
- removed joint ns1_left_inner_finger_joint
- removed joint ns1_left_inner_knuckle_joint
- removed joint ns1_left_outer_finger_joint
- removed joint ns1_panda_joint1
- removed joint ns1_panda_joint2
- removed joint ns1_panda_joint3
- removed joint ns1_panda_joint4
- removed joint ns1_panda_joint5
- removed joint ns1_panda_joint6
- removed joint ns1_panda_joint7
- removed joint ns1_panda_joint8
- removed joint ns1_panda_robotiq_attachment_joint
- removed joint ns1_panda_to_world
- removed joint ns1_rear_bumper
- removed joint ns1_right_inner_finger_joint
- removed joint ns1_right_inner_knuckle_joint
- removed joint ns1_right_outer_finger_joint
- removed joint ns1_right_outer_knuckle_joint
- removed joint ns1_top_chassis_joint
- removed joint ns1_top_plate_front_joint
- removed joint ns1_top_plate_joint
- removed joint ns1_top_plate_rear_joint
- removed joint ns1_user_rail
- added joint base_footprint_joint: type fixed, parent base_link, child base_footprint, origin xyz=0 0 -0.13228 rpy=0 0 0
- added joint finger_joint: type fixed, parent robotiq_85_base_link, child left_outer_knuckle, origin xyz=0.0306011444260539 0 0.0627920162695395 rpy=0 0 0, axis 0 -1 0, limit lower=0 upper=0.725 effort=1000 velocity=2.0
- added joint front_bumper: type fixed, parent base_link, child front_bumper_link, origin xyz=0.48 0 0.091 rpy=0 0 0
- added joint husky_front_left_wheel: type revolute, parent base_link, child husky_front_left_wheel_link, origin xyz=0.0 0.2854 0.03282 rpy=0 0 0, axis 0 -1 0, limit lower=-1000 upper=1000 effort=1000 velocity=100
- added joint husky_front_right_wheel: type revolute, parent base_link, child husky_front_right_wheel_link, origin xyz=0.0 -0.2854 0.03282 rpy=0 0 0, axis 0 1 0, limit lower=-1000 upper=1000 effort=1000 velocity=100
- added joint imu_joint: type fixed, parent base_link, child imu_link, origin xyz=0.19 0 0.149 rpy=0 -1.5708 3.1416
- added joint inertial_joint: type fixed, parent base_link, child inertial_link, origin xyz=0 0 0 rpy=0 0 0
- added joint left_inner_finger_joint: type fixed, parent left_inner_knuckle, child left_inner_finger, origin xyz=0.034585310861294 0 0.0454970193817975 rpy=0 0 0, axis 0 -1 0, limit lower=0 upper=0.8757 effort=1000 velocity=2.0, mimic joint=finger_joint multiplier=-1 offset=0
- added joint left_inner_knuckle_joint: type fixed, parent robotiq_85_base_link, child left_inner_knuckle, origin xyz=0.0127000000001501 0 0.0693074999999639 rpy=0 0 0, axis 0 -1 0, limit lower=0 upper=0.8757 effort=1000 velocity=2.0, mimic joint=finger_joint multiplier=1 offset=0
- added joint left_outer_finger_joint: type fixed, parent left_outer_knuckle, child left_outer_finger, origin xyz=0.0316910442266543 0 -0.00193396375724605 rpy=0 0 0, axis 0 -1 0
- added joint panda_joint1: type revolute, parent panda_link0, child panda_link1, origin xyz=0 0 0.333 rpy=0 0 0, axis 0 0 1, limit lower=-2.8973 upper=2.8973 effort=87 velocity=2.1750
- added joint panda_joint2: type revolute, parent panda_link1, child panda_link2, origin xyz=0 0 0 rpy=-1.57079632679 0 0, axis 0 0 1, limit lower=-1.7628 upper=1.7628 effort=87 velocity=2.1750
- added joint panda_joint3: type revolute, parent panda_link2, child panda_link3, origin xyz=0 -0.316 0 rpy=1.57079632679 0 0, axis 0 0 1, limit lower=-2.8973 upper=2.8973 effort=87 velocity=2.1750
- added joint panda_joint4: type revolute, parent panda_link3, child panda_link4, origin xyz=0.0825 0 0 rpy=1.57079632679 0 0, axis 0 0 1, limit lower=-3.0718 upper=-0.0698 effort=87 velocity=2.1750
- added joint panda_joint5: type revolute, parent panda_link4, child panda_link5, origin xyz=-0.0825 0.384 0 rpy=-1.57079632679 0 0, axis 0 0 1, limit lower=-2.8973 upper=2.8973 effort=12 velocity=2.6100
- added joint panda_joint6: type revolute, parent panda_link5, child panda_link6, origin xyz=0 0 0 rpy=1.57079632679 0 0, axis 0 0 1, limit lower=-0.0175 upper=3.7525 effort=12 velocity=2.6100
- added joint panda_joint7: type revolute, parent panda_link6, child panda_link7, origin xyz=0.088 0 0 rpy=1.57079632679 0 0, axis 0 0 1, limit lower=-2.8973 upper=2.8973 effort=12 velocity=2.6100
- added joint panda_joint8: type fixed, parent panda_link7, child panda_link8, origin xyz=0 0 0.107 rpy=0 0 0, axis 0 0 0
- added joint panda_robotiq_attachment_joint: type fixed, parent panda_link8, child robotiq_85_base_link, origin xyz=0 0 0 rpy=0 0 1.5707963268, axis 0 0 0
- added joint panda_to_world: type fixed, parent base_link, child panda_link0, origin xyz=0.35 0 0.25 rpy=0 0 0
- added joint rear_bumper: type fixed, parent base_link, child rear_bumper_link, origin xyz=-0.48 0 0.091 rpy=0 0 3.14159
- added joint right_inner_finger_joint: type fixed, parent right_inner_knuckle, child right_inner_finger, origin xyz=0.0341060475457406 0 0.0458573878541688 rpy=0 0 0, axis 0 1 0, limit lower=0 upper=0.8757 effort=1000 velocity=2.0, mimic joint=finger_joint multiplier=1 offset=0
- added joint right_inner_knuckle_joint: type fixed, parent robotiq_85_base_link, child right_inner_knuckle, origin xyz=-0.0126999999998499 0 0.0693075000000361 rpy=0 0 3.14159265358979, axis 0 1 0, limit lower=0 upper=0.8757 effort=1000 velocity=2.0, mimic joint=finger_joint multiplier=-1 offset=0
- added joint right_outer_finger_joint: type fixed, parent right_outer_knuckle, child right_outer_finger, origin xyz=0.0317095909367246 0 -0.0016013564954687 rpy=0 0 0, axis 0 1 0
- added joint right_outer_knuckle_joint: type fixed, parent robotiq_85_base_link, child right_outer_knuckle, origin xyz=-0.0306011444258893 0 0.0627920162695395 rpy=0 0 3.14159265358979, axis 0 1 0, limit lower=0 upper=0.8757 effort=1000 velocity=2.0, mimic joint=finger_joint multiplier=-1 offset=0
- added joint top_chassis_joint: type fixed, parent base_link, child top_chassis_link
- added joint top_plate_front_joint: type fixed, parent top_plate_link, child top_plate_front_link, origin xyz=0.36367 0 0.00639 rpy=0 0 0
- added joint top_plate_joint: type fixed, parent base_link, child top_plate_link, origin xyz=0.0812 0 0.245 rpy=0 0 0
- added joint top_plate_rear_joint: type fixed, parent top_plate_link, child top_plate_rear_link, origin xyz=-0.36633 0 0.00639 rpy=0 0 0
- added joint user_rail: type fixed, parent base_link, child user_rail_link, origin xyz=0.272 0 0.245 rpy=0 0 0
- added joint v_t_joint: type revolute, parent v_t_link, child base_link, origin xyz=0 0 0.0 rpy=0 0 0, axis 0 0 1, limit lower=-6.24 upper=6.24 effort=1000.0 velocity=10000.0
- added joint v_x_joint: type prismatic, parent v_x_link, child v_y_link, origin xyz=0 0 0.0 rpy=0 0 0, axis 1 0 0, limit lower=-10000.0 upper=-10000.0 effort=1000.0 velocity=10000.0
- added joint v_y_joint: type prismatic, parent v_y_link, child v_t_link, origin xyz=0 0 0.0 rpy=0 0 0, axis 0 1 0, limit lower=-10000.0 upper=-10000.0 effort=1000.0 velocity=10000.0
