Commit message: update simul robot:

File: franka_panda_description/franka_single/panda_arm_hand_l.urdf (robot description, URDF)
Before this commit: robot panda, 10 links, 9 joints
Links:
- removed link base_link
- added link panda_hand, mass 0.73; collision mesh filename=package://franka_panda_description/meshes/collision/hand.stl; visual mesh filename=package://franka_panda_description/meshes/visual/hand.dae
- added link panda_leftfinger, mass 0.1; collision mesh filename=package://franka_panda_description/meshes/collision/finger.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; visual mesh filename=package://franka_panda_description/meshes/visual/finger.dae
- added link panda_rightfinger, mass 0.1; collision mesh filename=package://franka_panda_description/meshes/collision/finger.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; visual mesh filename=package://franka_panda_description/meshes/visual/finger.dae
- added link world
- link panda_link8: mass 0.0 -> 0.01
Joints:
- removed joint l_panda_joint1
- removed joint l_panda_joint2
- removed joint l_panda_joint3
- removed joint l_panda_joint4
- removed joint l_panda_joint5
- removed joint l_panda_joint6
- removed joint l_panda_joint7
- removed joint l_panda_joint8
- removed joint l_panda_to_world
- added joint panda_finger_joint1: type fixed, parent panda_hand, child panda_leftfinger, origin xyz=0 0 0.0584 rpy=0 0 0, axis 0 1 0, limit lower=0.0 upper=0.04 effort=20 velocity=0.2
- added joint panda_finger_joint2: type fixed, parent panda_hand, child panda_rightfinger, origin xyz=0 0 0.0584 rpy=0 0 0, axis 0 -1 0, limit lower=0.0 upper=0.04 effort=20 velocity=0.2, mimic joint=panda_finger_joint1
- added joint panda_hand_joint: type fixed, parent panda_link8, child panda_hand, origin xyz=0.0 0 0 rpy=0 0 -0.785398163397
- added joint panda_joint1: type revolute, parent panda_link0, child panda_link1, origin xyz=0 0 0.333 rpy=0 0 0, axis 0 0 1, limit lower=-2.8973 upper=2.8973 effort=87 velocity=2.1750
- added joint panda_joint2: type revolute, parent panda_link1, child panda_link2, origin xyz=0 0 0 rpy=-1.57079632679 0 0, axis 0 0 1, limit lower=-1.7628 upper=1.7628 effort=87 velocity=2.1750
- added joint panda_joint3: type revolute, parent panda_link2, child panda_link3, origin xyz=0 -0.316 0 rpy=1.57079632679 0 0, axis 0 0 1, limit lower=-2.8973 upper=2.8973 effort=87 velocity=2.1750
- added joint panda_joint4: type revolute, parent panda_link3, child panda_link4, origin xyz=0.0825 0 0 rpy=1.57079632679 0 0, axis 0 0 1, limit lower=-3.0718 upper=-0.0698 effort=87 velocity=2.1750
- added joint panda_joint5: type revolute, parent panda_link4, child panda_link5, origin xyz=-0.0825 0.384 0 rpy=-1.57079632679 0 0, axis 0 0 1, limit lower=-2.8973 upper=2.8973 effort=12 velocity=2.6100
- added joint panda_joint6: type revolute, parent panda_link5, child panda_link6, origin xyz=0 0 0 rpy=1.57079632679 0 0, axis 0 0 1, limit lower=-0.0175 upper=3.7525 effort=12 velocity=2.6100
- added joint panda_joint7: type revolute, parent panda_link6, child panda_link7, origin xyz=0.088 0 0 rpy=1.57079632679 0 0, axis 0 0 1, limit lower=-2.8973 upper=2.8973 effort=12 velocity=2.6100
- added joint panda_joint8: type fixed, parent panda_link7, child panda_link8, origin xyz=0 0 0.107 rpy=0 0 0, axis 0 0 0
- added joint panda_to_world: type fixed, parent world, child panda_link0, origin xyz=-1 0 0 rpy=0 0 0

File: franka_panda_description/franka_single/panda_arm_hand_l_rviz.urdf (robot description, URDF)
Before this commit: robot panda, 10 links, 9 joints
Links:
- removed link base_link
- added link panda_hand, mass 0.73; collision mesh filename=package://franka_panda_description/meshes/collision/hand.stl; visual mesh filename=package://franka_panda_description/meshes/visual/hand.dae
- added link panda_leftfinger, mass 0.1; collision mesh filename=package://franka_panda_description/meshes/collision/finger.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; visual mesh filename=package://franka_panda_description/meshes/visual/finger.dae
- added link panda_rightfinger, mass 0.1; collision mesh filename=package://franka_panda_description/meshes/collision/finger.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; visual mesh filename=package://franka_panda_description/meshes/visual/finger.dae
- added link world
- link panda_link8: mass 0.0 -> 0.01
Joints:
- removed joint l_panda_joint1
- removed joint l_panda_joint2
- removed joint l_panda_joint3
- removed joint l_panda_joint4
- removed joint l_panda_joint5
- removed joint l_panda_joint6
- removed joint l_panda_joint7
- removed joint l_panda_joint8
- removed joint l_panda_to_world
- added joint panda_finger_joint1: type prismatic, parent panda_hand, child panda_leftfinger, origin xyz=0 0 0.0584 rpy=0 0 0, axis 0 1 0, limit lower=0.0 upper=0.04 effort=20 velocity=0.2
- added joint panda_finger_joint2: type prismatic, parent panda_hand, child panda_rightfinger, origin xyz=0 0 0.0584 rpy=0 0 0, axis 0 -1 0, limit lower=0.0 upper=0.04 effort=20 velocity=0.2, mimic joint=panda_finger_joint1
- added joint panda_hand_joint: type fixed, parent panda_link8, child panda_hand, origin xyz=0.0 0 0 rpy=0 0 -0.785398163397
- added joint panda_joint1: type revolute, parent panda_link0, child panda_link1, origin xyz=0 0 0.333 rpy=0 0 0, axis 0 0 1, limit lower=-2.8973 upper=2.8973 effort=87 velocity=2.1750
- added joint panda_joint2: type revolute, parent panda_link1, child panda_link2, origin xyz=0 0 0 rpy=-1.57079632679 0 0, axis 0 0 1, limit lower=-1.7628 upper=1.7628 effort=87 velocity=2.1750
- added joint panda_joint3: type revolute, parent panda_link2, child panda_link3, origin xyz=0 -0.316 0 rpy=1.57079632679 0 0, axis 0 0 1, limit lower=-2.8973 upper=2.8973 effort=87 velocity=2.1750
- added joint panda_joint4: type revolute, parent panda_link3, child panda_link4, origin xyz=0.0825 0 0 rpy=1.57079632679 0 0, axis 0 0 1, limit lower=-3.0718 upper=-0.0698 effort=87 velocity=2.1750
- added joint panda_joint5: type revolute, parent panda_link4, child panda_link5, origin xyz=-0.0825 0.384 0 rpy=-1.57079632679 0 0, axis 0 0 1, limit lower=-2.8973 upper=2.8973 effort=12 velocity=2.6100
- added joint panda_joint6: type revolute, parent panda_link5, child panda_link6, origin xyz=0 0 0 rpy=1.57079632679 0 0, axis 0 0 1, limit lower=-0.0175 upper=3.7525 effort=12 velocity=2.6100
- added joint panda_joint7: type revolute, parent panda_link6, child panda_link7, origin xyz=0.088 0 0 rpy=1.57079632679 0 0, axis 0 0 1, limit lower=-2.8973 upper=2.8973 effort=12 velocity=2.6100
- added joint panda_joint8: type fixed, parent panda_link7, child panda_link8, origin xyz=0 0 0.107 rpy=0 0 0, axis 0 0 0
- added joint panda_to_world: type fixed, parent world, child panda_link0, origin xyz=-1 0 0 rpy=0 0 0

Commit message: modify world position (0,0,0)

File: franka_panda_description/franka_single/panda_arm_hand_l.urdf (robot description, URDF)
Before this commit: robot panda, 13 links, 12 joints
Joints:
- joint panda_to_world: origin xyz=-1 0 0 rpy=0 0 0 -> xyz=0 0 0 rpy=0 0 0

File: franka_panda_description/franka_single/panda_arm_hand_l_rviz.urdf (robot description, URDF)
Before this commit: robot panda, 13 links, 12 joints
Joints:
- joint panda_to_world: origin xyz=-1 0 0 rpy=0 0 0 -> xyz=0 0 0 rpy=0 0 0
