Commit message: modify urdf naming

File: franka_panda_description/franka_single/fr3_arm_2f_85_d435.urdf (robot description, URDF)
Before this commit: robot panda, 19 links, 18 joints
Links:
- added link camera_bottom_screw_frame
- added link camera_color_frame
- added link camera_color_optical_frame
- added link camera_depth_frame
- added link camera_depth_optical_frame
- added link camera_jig_link
- added link camera_left_ir_frame
- added link camera_left_ir_optical_frame
- added link camera_link, mass 0.072; collision box size=0.02505 0.09 0.025; visual mesh filename=package://realsense2_description/meshes/d435.dae
- added link camera_right_ir_frame
- added link camera_right_ir_optical_frame
Joints:
- added joint camera_color_joint: type fixed, parent camera_depth_frame, child camera_color_frame, origin xyz=0 0.015 0 rpy=0 0 0
- added joint camera_color_optical_joint: type fixed, parent camera_color_frame, child camera_color_optical_frame, origin xyz=0 0 0 rpy=-1.57079632679 0 -1.57079632679
- added joint camera_depth_joint: type fixed, parent camera_link, child camera_depth_frame, origin xyz=0 0 0 rpy=0 0 0
- added joint camera_depth_optical_joint: type fixed, parent camera_depth_frame, child camera_depth_optical_frame, origin xyz=0 0 0 rpy=-1.57079632679 0 -1.57079632679
- added joint camera_jig_joint: type fixed, parent robotiq_85_base_link, child camera_jig_link, origin xyz=0.0 0 0.0 rpy=0.0 0.0 0
- added joint camera_joint: type fixed, parent camera_jig_link, child camera_bottom_screw_frame, origin xyz=0.0 -0.09 0.085 rpy=3.14 -1.57 -1.57
- added joint camera_left_ir_joint: type fixed, parent camera_depth_frame, child camera_left_ir_frame, origin xyz=0 0.0 0 rpy=0 0 0
- added joint camera_left_ir_optical_joint: type fixed, parent camera_left_ir_frame, child camera_left_ir_optical_frame, origin xyz=0 0 0 rpy=-1.57079632679 0 -1.57079632679
- added joint camera_link_joint: type fixed, parent camera_bottom_screw_frame, child camera_link, origin xyz=0 0.0175 0.0125 rpy=0 0 0
- added joint camera_right_ir_joint: type fixed, parent camera_depth_frame, child camera_right_ir_frame, origin xyz=0 -0.05 0 rpy=0 0 0
- added joint camera_right_ir_optical_joint: type fixed, parent camera_right_ir_frame, child camera_right_ir_optical_frame, origin xyz=0 0 0 rpy=-1.57079632679 0 -1.57079632679
- joint finger_joint: type revolute -> fixed
- joint left_inner_finger_joint: type revolute -> fixed
- joint left_inner_knuckle_joint: type revolute -> fixed
- joint panda_robotiq_attachment_joint: origin xyz=0 0 0 rpy=0 0 1.5707963268 -> xyz=0 0 0 rpy=0 0 0.0
- joint right_inner_finger_joint: type revolute -> fixed
- joint right_inner_knuckle_joint: type revolute -> fixed
- joint right_outer_knuckle_joint: type revolute -> fixed

File: franka_panda_description/franka_single/fr3_arm_2f_85_d435_rviz.urdf (robot description, URDF)
Before this commit: robot panda, 19 links, 18 joints
Links:
- added link camera_bottom_screw_frame
- added link camera_color_frame
- added link camera_color_optical_frame
- added link camera_depth_frame
- added link camera_depth_optical_frame
- added link camera_jig_link
- added link camera_left_ir_frame
- added link camera_left_ir_optical_frame
- added link camera_link, mass 0.072; collision box size=0.02505 0.09 0.025; visual mesh filename=package://realsense2_description/meshes/d435.dae
- added link camera_right_ir_frame
- added link camera_right_ir_optical_frame
Joints:
- added joint camera_color_joint: type fixed, parent camera_depth_frame, child camera_color_frame, origin xyz=0 0.015 0 rpy=0 0 0
- added joint camera_color_optical_joint: type fixed, parent camera_color_frame, child camera_color_optical_frame, origin xyz=0 0 0 rpy=-1.57079632679 0 -1.57079632679
- added joint camera_depth_joint: type fixed, parent camera_link, child camera_depth_frame, origin xyz=0 0 0 rpy=0 0 0
- added joint camera_depth_optical_joint: type fixed, parent camera_depth_frame, child camera_depth_optical_frame, origin xyz=0 0 0 rpy=-1.57079632679 0 -1.57079632679
- added joint camera_jig_joint: type fixed, parent robotiq_85_base_link, child camera_jig_link, origin xyz=0.0 0 0.0 rpy=0.0 0.0 0
- added joint camera_joint: type fixed, parent camera_jig_link, child camera_bottom_screw_frame, origin xyz=0.0 -0.09 0.085 rpy=3.14 -1.57 -1.57
- added joint camera_left_ir_joint: type fixed, parent camera_depth_frame, child camera_left_ir_frame, origin xyz=0 0.0 0 rpy=0 0 0
- added joint camera_left_ir_optical_joint: type fixed, parent camera_left_ir_frame, child camera_left_ir_optical_frame, origin xyz=0 0 0 rpy=-1.57079632679 0 -1.57079632679
- added joint camera_link_joint: type fixed, parent camera_bottom_screw_frame, child camera_link, origin xyz=0 0.0175 0.0125 rpy=0 0 0
- added joint camera_right_ir_joint: type fixed, parent camera_depth_frame, child camera_right_ir_frame, origin xyz=0 -0.05 0 rpy=0 0 0
- added joint camera_right_ir_optical_joint: type fixed, parent camera_right_ir_frame, child camera_right_ir_optical_frame, origin xyz=0 0 0 rpy=-1.57079632679 0 -1.57079632679
- joint panda_robotiq_attachment_joint: origin xyz=0 0 0 rpy=0 0 1.5707963268 -> xyz=0 0 0 rpy=0 0 0.0

File: franka_panda_description/franka_single/panda_arm_2f_85.urdf (robot description, URDF)
Before this commit: robot panda, 19 links, 18 joints
Links:
- link robotiq_85_base_link: mass 0.30915 -> 0.79501

File: franka_panda_description/franka_single/panda_arm_hand_d435.urdf (robot description, URDF)
Before this commit: robot panda, 23 links, 22 joints
Links:
- link camera_link: mass 0.564 -> 0.072
Joints:
- joint panda_finger_joint1: type prismatic -> fixed
- joint panda_finger_joint2: type prismatic -> fixed

Commit message: add moveit application w/ fr3

File: franka_panda_description/franka_single/fr3_arm_2f_85_d435.urdf (robot description, URDF)
Before this commit: robot panda, 30 links, 29 joints
Joints:
- joint camera_joint: origin xyz=0.0 -0.09 0.085 rpy=3.14 -1.57 -1.57 -> xyz=0.0 0.065 0.055 rpy=3.14 -1.57 1.57

File: franka_panda_description/franka_single/fr3_arm_2f_85_d435_moveit.urdf (robot description, URDF)
Before this commit: robot panda, 30 links, 29 joints
Links:
- removed link camera_bottom_screw_frame
- removed link camera_color_frame
- removed link camera_color_optical_frame
- removed link camera_depth_frame
- removed link camera_depth_optical_frame
- removed link camera_jig_link
- removed link camera_left_ir_frame
- removed link camera_left_ir_optical_frame
- removed link camera_link
- removed link camera_right_ir_frame
- removed link camera_right_ir_optical_frame
- removed link left_inner_finger
- removed link left_inner_knuckle
- removed link left_outer_finger
- removed link left_outer_knuckle
- removed link panda_link0
- removed link panda_link1
- removed link panda_link2
- removed link panda_link3
- removed link panda_link4
- removed link panda_link5
- removed link panda_link6
- removed link panda_link7
- removed link panda_link8
- removed link right_inner_finger
- removed link right_inner_knuckle
- removed link right_outer_finger
- removed link right_outer_knuckle
- removed link robotiq_85_base_link
- added link m_camera_bottom_screw_frame
- added link m_camera_color_frame
- added link m_camera_color_optical_frame
- added link m_camera_depth_frame
- added link m_camera_depth_optical_frame
- added link m_camera_jig_link
- added link m_camera_left_ir_frame
- added link m_camera_left_ir_optical_frame
- added link m_camera_link, mass 0.072; collision box size=0.02505 0.09 0.025; visual mesh filename=package://realsense2_description/meshes/d435.dae
- added link m_camera_right_ir_frame
- added link m_camera_right_ir_optical_frame
- added link m_left_inner_finger, mass 0.00724255346165745; collision mesh filename=package://kimm_robotiq_2f_85_description/meshes_aprice/inne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; visual mesh filename=package://kimm_robotiq_2f_85_description/meshes_aprice/inne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
- added link m_left_inner_knuckle, mass 0.0110930853895903; collision mesh filename=package://kimm_robotiq_2f_85_description/meshes_aprice/inne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; visual mesh filename=package://kimm_robotiq_2f_85_description/meshes_aprice/inne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
- added link m_left_outer_finger, mass 0.0273093985570947; collision mesh filename=package://kimm_robotiq_2f_85_description/meshes_aprice/oute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; visual mesh filename=package://kimm_robotiq_2f_85_description/meshes_aprice/oute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
- added link m_left_outer_knuckle, mass 0.00684838849434396; collision mesh filename=package://kimm_robotiq_2f_85_description/meshes_aprice/oute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; visual mesh filename=package://kimm_robotiq_2f_85_description/meshes_aprice/oute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
- added link m_panda_link0; collision mesh filename=package://franka_panda_description/meshes/collision/link0.s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; visual mesh filename=package://franka_panda_description/meshes/visual/link0.dae
- added link m_panda_link1, mass 4.970684; collision mesh filename=package://franka_panda_description/meshes/collision/link1.s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; visual mesh filename=package://franka_panda_description/meshes/visual/link1.dae
- added link m_panda_link2, mass 0.646926; collision mesh filename=package://franka_panda_description/meshes/collision/link2.s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; visual mesh filename=package://franka_panda_description/meshes/visual/link2.dae
- added link m_panda_link3, mass 3.228604; collision mesh filename=package://franka_panda_description/meshes/collision/link3.s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; visual mesh filename=package://franka_panda_description/meshes/visual/link3.dae
- added link m_panda_link4, mass 3.587895; collision mesh filename=package://franka_panda_description/meshes/collision/link4.s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; visual mesh filename=package://franka_panda_description/meshes/visual/link4.dae
- added link m_panda_link5, mass 1.225946; collision mesh filename=package://franka_panda_description/meshes/collision/link5.s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; visual mesh filename=package://franka_panda_description/meshes/visual/link5.dae
- added link m_panda_link6, mass 1.666555; collision mesh filename=package://franka_panda_description/meshes/collision/link6.s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; visual mesh filename=package://franka_panda_description/meshes/visual/link6.dae
- added link m_panda_link7, mass 7.35522e-01; collision mesh filename=package://franka_panda_description/meshes/collision/link7.s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; visual mesh filename=package://franka_panda_description/meshes/visual/link7.dae
- added link m_panda_link8, mass 0.01
- added link m_right_inner_finger, mass 0.00724255346165744; collision mesh filename=package://kimm_robotiq_2f_85_description/meshes_aprice/inne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; visual mesh filename=package://kimm_robotiq_2f_85_description/meshes_aprice/inne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
- added link m_right_inner_knuckle, mass 0.0110930853895903; collision mesh filename=package://kimm_robotiq_2f_85_description/meshes_aprice/inne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; visual mesh filename=package://kimm_robotiq_2f_85_description/meshes_aprice/inne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
- added link m_right_outer_finger, mass 0.0273093985570947; collision mesh filename=package://kimm_robotiq_2f_85_description/meshes_aprice/oute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; visual mesh filename=package://kimm_robotiq_2f_85_description/meshes_aprice/oute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
- added link m_right_outer_knuckle, mass 0.00684838849401352; collision mesh filename=package://kimm_robotiq_2f_85_description/meshes_aprice/oute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; visual mesh filename=package://kimm_robotiq_2f_85_description/meshes_aprice/oute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
- added link m_robotiq_85_base_link, mass 0.79501; collision mesh filename=package://kimm_robotiq_2f_85_description/meshes_aprice/robo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; visual mesh filename=package://kimm_robotiq_2f_85_description/meshes_aprice/robo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
Joints:
- joint camera_color_joint: child camera_color_frame -> m_camera_color_frame; parent camera_depth_frame -> m_camera_depth_frame
- joint camera_color_optical_joint: child camera_color_optical_frame -> m_camera_color_optical_frame; parent camera_color_frame -> m_camera_color_frame
- joint camera_depth_joint: child camera_depth_frame -> m_camera_depth_frame; parent camera_link -> m_camera_link
- joint camera_depth_optical_joint: child camera_depth_optical_frame -> m_camera_depth_optical_frame; parent camera_depth_frame -> m_camera_depth_frame
- joint camera_jig_joint: child camera_jig_link -> m_camera_jig_link; parent robotiq_85_base_link -> m_robotiq_85_base_link
- joint camera_joint: child camera_bottom_screw_frame -> m_camera_bottom_screw_frame; parent camera_jig_link -> m_camera_jig_link
- joint camera_left_ir_joint: child camera_left_ir_frame -> m_camera_left_ir_frame; parent camera_depth_frame -> m_camera_depth_frame
- joint camera_left_ir_optical_joint: child camera_left_ir_optical_frame -> m_camera_left_ir_optical_frame; parent camera_left_ir_frame -> m_camera_left_ir_frame
- joint camera_link_joint: child camera_link -> m_camera_link; parent camera_bottom_screw_frame -> m_camera_bottom_screw_frame
- joint camera_right_ir_joint: child camera_right_ir_frame -> m_camera_right_ir_frame; parent camera_depth_frame -> m_camera_depth_frame
- joint camera_right_ir_optical_joint: child camera_right_ir_optical_frame -> m_camera_right_ir_optical_frame; parent camera_right_ir_frame -> m_camera_right_ir_frame
- joint finger_joint: child left_outer_knuckle -> m_left_outer_knuckle; parent robotiq_85_base_link -> m_robotiq_85_base_link; type revolute -> fixed
- joint left_inner_finger_joint: child left_inner_finger -> m_left_inner_finger; parent left_inner_knuckle -> m_left_inner_knuckle; type revolute -> fixed
- joint left_inner_knuckle_joint: child left_inner_knuckle -> m_left_inner_knuckle; parent robotiq_85_base_link -> m_robotiq_85_base_link; type revolute -> fixed
- joint left_outer_finger_joint: child left_outer_finger -> m_left_outer_finger; parent left_outer_knuckle -> m_left_outer_knuckle
- joint panda_joint1: child panda_link1 -> m_panda_link1; parent panda_link0 -> m_panda_link0
- joint panda_joint2: child panda_link2 -> m_panda_link2; parent panda_link1 -> m_panda_link1
- joint panda_joint3: child panda_link3 -> m_panda_link3; parent panda_link2 -> m_panda_link2
- joint panda_joint4: child panda_link4 -> m_panda_link4; parent panda_link3 -> m_panda_link3
- joint panda_joint5: child panda_link5 -> m_panda_link5; parent panda_link4 -> m_panda_link4
- joint panda_joint6: child panda_link6 -> m_panda_link6; parent panda_link5 -> m_panda_link5
- joint panda_joint7: child panda_link7 -> m_panda_link7; parent panda_link6 -> m_panda_link6
- joint panda_joint8: child panda_link8 -> m_panda_link8; parent panda_link7 -> m_panda_link7
- joint panda_robotiq_attachment_joint: child robotiq_85_base_link -> m_robotiq_85_base_link; parent panda_link8 -> m_panda_link8
- joint panda_to_world: child panda_link0 -> m_panda_link0
- joint right_inner_finger_joint: child right_inner_finger -> m_right_inner_finger; parent right_inner_knuckle -> m_right_inner_knuckle; type revolute -> fixed
- joint right_inner_knuckle_joint: child right_inner_knuckle -> m_right_inner_knuckle; parent robotiq_85_base_link -> m_robotiq_85_base_link; type revolute -> fixed
- joint right_outer_finger_joint: child right_outer_finger -> m_right_outer_finger; parent right_outer_knuckle -> m_right_outer_knuckle
- joint right_outer_knuckle_joint: child right_outer_knuckle -> m_right_outer_knuckle; parent robotiq_85_base_link -> m_robotiq_85_base_link; type revolute -> fixed
